Commit message: Added basic driving function(WIP)

File: description/robot_core.xacro (robot description, xacro)
@@ -43,4 +43,8 @@
         </xacro:inertial_box>
     </link>
+    <gazebo reference="chassis">
+        <material>white</material>
+        <static>false</static>
+    </gazebo>
     <!-- TOP LEFT WHEEL LINK-->
     <joint name="top_left_wheel_joint" type="continuous">
@@ -66,4 +70,7 @@
         </xacro:inertial_cylinder>
     </link>
+    <gazebo reference="top_left_wheel">
+        <material>blue</material>
+    </gazebo>
     <!-- TOP RIGHT WHEEL LINK-->
     <joint name="top_right_wheel_joint" type="continuous">
@@ -89,4 +96,7 @@
         </xacro:inertial_cylinder>
     </link>
+    <gazebo reference="top_right_wheel">
+        <material>blue</material>
+    </gazebo>
     <!-- BOTTOM LEFT WHEEL LINK-->
     <joint name="bottom_left_wheel_joint" type="continuous">
@@ -112,4 +122,7 @@
         </xacro:inertial_cylinder>
     </link>
+    <gazebo reference="bottom_left_wheel">
+        <material>blue</material>
+    </gazebo>
     <!-- BOTTOM RIGHT WHEEL LINK-->
     <joint name="bottom_right_wheel_joint" type="continuous">
@@ -135,3 +148,6 @@
         </xacro:inertial_cylinder>
     </link>
+    <gazebo reference="bottom_right_wheel">
+        <material>blue</material>
+    </gazebo>
 </robot>
