Commit message: Added controller files

File: description/camera.xacro (robot description, xacro)
@@ -52,5 +52,5 @@
                 <update_rate>20</update_rate>
                 <visualize>true</visualize>
-                <topic>camera/image</topic>
+                <topic>camera/image_raw</topic>
             </sensor>
         </gazebo>

File: description/robot.urdf.xacro (robot description, xacro)
@@ -3,6 +3,7 @@
     <xacro:include filename="robot_core.xacro"/>
     <!-- <xacro:include filename="gazebo_control.xacro"/> -->
-    <!-- <xacro:include filename="camera.xacro"/> -->
-    <xacro:include filename="lidar.xacro"/>
+    <xacro:include filename="ros2_control.xacro"/>
+    <xacro:include filename="camera.xacro"/>
+    <!-- <xacro:include filename="lidar.xacro"/> -->
     <!-- <xacro:include filename="ros2_control.xacro"/> -->
 </robot>

File: description/ros2_control.xacro (robot description, xacro)
@@ -1,10 +1,12 @@
-<!-- <?xml version="1.0"?>
+<?xml version="1.0"?>
 <robot xmlns:xacro="http://www.ros.org/wiki/xacro" name="robot">
-    <xacro:unless value="$(arg sim_mode)">
+    <!-- <xacro:unless value="$(arg sim_mode)">
         <ros2_control name="RealRobot" type="system">
             <hardware>
                 <plugin>diffdrive_arduino/DiffDriveArduinoHardware</plugin>
-                <param name="left_wheel_name">left_wheel_joint</param>
-                <param name="right_wheel_name">right_wheel_joint</param>
+                <param name="top_left_wheel_name">top_left_wheel_joint</param>
+                <param name="top_right_wheel_name">top_right_wheel_joint</param>
+                <param name="bottom_left_wheel_name">bottom_left_wheel_joint</param>
+                <param name="bottom_right_wheel_name">bottom_right_wheel_joint</param>
                 <param name="loop_rate">30</param>
                 <param name="device">/dev/ttyUSB0</param>
@@ -46,28 +48,44 @@
             </joint>
         </ros2_control>
-    </xacro:unless>
-    <xacro:if value="$(arg sim_mode)">
+    </xacro:unless> -->
+    <!-- <xacro:if value="$(arg sim_mode)"> -->
         <ros2_control name="GazeboSystem" type="system">
             <hardware>
                 <plugin>gz_ros2_control/GazeboSimSystem</plugin>
             </hardware>
-            <joint name="left_wheel_joint">
+            <joint name="top_left_wheel_joint">
                 <command_interface name="velocity">
                     <param name="min">-10</param>
                     <param name="max">10</param>
                 </command_interface>
+                <state_interface name="position"/>
                 <state_interface name="velocity"/>
-                <state_interface name="position"/>
             </joint>
-            <joint name="right_wheel_joint">
+            <joint name="bottom_left_wheel_joint">
                 <command_interface name="velocity">
                     <param name="min">-10</param>
                     <param name="max">10</param>
                 </command_interface>
+                <state_interface name="position"/>
                 <state_interface name="velocity"/>
+            </joint>
+            <joint name="top_right_wheel_joint">
+                <command_interface name="velocity">
+                    <param name="min">-10</param>
+                    <param name="max">10</param>
+                </command_interface>
                 <state_interface name="position"/>
+                <state_interface name="velocity"/>
+            </joint>
+            <joint name="bottom_right_wheel_joint">
+                <command_interface name="velocity">
+                    <param name="min">-10</param>
+                    <param name="max">10</param>
+                </command_interface>
+                <state_interface name="position"/>
+                <state_interface name="velocity"/>
             </joint>
         </ros2_control>
-    </xacro:if>
+    <!-- </xacro:if> -->
     <gazebo>
         <plugin name="gz_ros2_control::GazeboSimROS2ControlPlugin" filename="libgz_ros2_control-system.so">
@@ -76,3 +94,3 @@
         </plugin>
     </gazebo>
-</robot> -->
+</robot>
