Commit message: Added scan LiDAR function just in case necessary

File: description/lidar.xacro (robot description, xacro)
@@ -1,4 +1,5 @@
 <?xml version="1.0"?>
 <robot xmlns:xacro="http://www.ros.org/wiki/xacro" >
+    <!--CAMERA JOINT-->
     <joint name="camera_joint" type="fixed">
         <parent link="chassis_link"/>
@@ -20,4 +21,43 @@
     </joint>
     <link name="camera_link_optical"></link>
+    <!--LASER SCAN JOINT-->
+    <joint name="laser_joint" type="fixed">
+        <parent link="chassis_link"/>
+        <child link="laser_frame"/>
+        <origin xyz="0.4 0 0.18" rpy="0 0 0"/>
+    </joint>
+    <link name="laser_frame">
+        <visual>
+            <geometry>
+                <box size="0.05 0.25 0.045"/>
+            </geometry>
+            <material name="black"/>
+        </visual>
+    </link>
+    <!--LIDAR CAMERA-->
+    <!-- <gazebo reference="laser_frame">
+      <sensor name="laser" type="gpu_lidar">
+         <pose> 0 0 0 0 0 0 </pose>
+         <always_on>true</always_on>
+         <visualize>true</visualize>
+         <update_rate>20</update_rate>
+         <topic>scan</topic>
+         <gz_frame_id>laser_frame</gz_frame_id>
+         <lidar>
+            <scan>
+               <horizontal>
+                <samples>360</samples>
+                <min_angle>-0.6109</min_angle>
+                <max_angle>0.6109</max_angle>
+              </horizontal>
+            </scan>
+            <range>
+               <min>0.3</min>
+               <max>12</max>
+            </range>
+         </lidar>
+      </sensor>
+   </gazebo> -->
+    <!--RGBD DEPTH CAMERA-->
     <gazebo reference="camera_link">
     <sensor name="rgbd_camera" type="rgbd_camera">
@@ -41,4 +81,5 @@
     </sensor>
   </gazebo>
+    <!--REGULAR CAMERA-->
     <!-- <sensor name="camera" type="camera">
       <camera>
