Commit message: added models to simulate obj detection, will add working files tomorrow

File: description/robot.urdf.xacro (robot description, xacro)
@@ -4,6 +4,6 @@
     <!-- <xacro:include filename="gazebo_control.xacro"/> -->
     <xacro:include filename="ros2_control.xacro"/>
-    <!-- <xacro:include filename="camera.xacro"/> -->
-    <xacro:include filename="lidar.xacro"/>
+    <xacro:include filename="camera.xacro"/>
+    <!-- <xacro:include filename="lidar.xacro"/> -->
     <!-- <xacro:include filename="ros2_control.xacro"/> -->
 </robot>

File: description/robot_core.xacro (robot description, xacro)
@@ -8,8 +8,8 @@
     </material>
     <material name="green">
-        <color rgba="0 1 0 1"/>
+        <color rgba="0 0.6 0 1"/>
     </material>
-    <material name="red">
-        <color rgba="1 0 0 1"/>
+    <material name="yellow">
+        <color rgba="0.8 0.8 0 1"/>
     </material>
     <material name="blue">
